Commit message: Fix dog movement by restoring realistic physics parameters
Root cause: Effort limit was increased to 1.0 Nm (7x real servo torque)
with very low damping/friction (0.01), causing unstable joint behavior.

Changes:
- Effort limit: 1.0 Nm → 0.15 Nm (matches real servo: 0.127-0.137 Nm)
- Damping: 0.01 → 0.5 (realistic joint resistance)
- Friction: 0.01 → 0.5 (realistic joint resistance)

Physics rationale:
- Real SunFounder SF006FM servo: 0.127-0.137 Nm stall torque
- Higher damping/friction prevents overshoot and provides stability
- 0.15 Nm effort limit allows realistic sim-to-real transfer

This restores realistic simulation parameters as documented in CLAUDE.md.
The robot should now move smoothly and predictably.

Fixes regression introduced in commit 2971cdd where effort was increased
to 1.0 Nm, breaking movement that was working at commit 68d721c.

File: pidog_description/urdf/pidog.urdf (robot description, URDF)
Before this commit: robot PiDog, 31 links, 30 joints
Joints:
- joint back_left_leg_b_to_a: limit lower=-1.57 upper=1.57 effort=1.0 velocity=7.0 -> lower=-1.57 upper=1.57 effort=0.15 velocity=7.0
- joint back_right_leg_b_to_a: limit lower=-1.57 upper=1.57 effort=1.0 velocity=7.0 -> lower=-1.57 upper=1.57 effort=0.15 velocity=7.0
- joint body_to_back_left_leg_b: limit lower=-1.57 upper=1.57 effort=1.0 velocity=7.0 -> lower=-1.57 upper=1.57 effort=0.15 velocity=7.0
- joint body_to_back_right_leg_b: limit lower=-1.57 upper=1.57 effort=1.0 velocity=7.0 -> lower=-1.57 upper=1.57 effort=0.15 velocity=7.0
- joint body_to_front_left_leg_b: limit lower=-1.57 upper=1.57 effort=1.0 velocity=7.0 -> lower=-1.57 upper=1.57 effort=0.15 velocity=7.0
- joint body_to_front_right_leg_b: limit lower=-1.57 upper=1.57 effort=1.0 velocity=7.0 -> lower=-1.57 upper=1.57 effort=0.15 velocity=7.0
- joint front_left_leg_b_to_a: limit lower=-1.57 upper=1.57 effort=1.0 velocity=7.0 -> lower=-1.57 upper=1.57 effort=0.15 velocity=7.0
- joint front_right_leg_b_to_a: limit lower=-1.57 upper=1.57 effort=1.0 velocity=7.0 -> lower=-1.57 upper=1.57 effort=0.15 velocity=7.0
- joint motor_8_to_tail: limit lower=-1.57 upper=1.57 effort=1.0 velocity=7.0 -> lower=-1.57 upper=1.57 effort=0.15 velocity=7.0

Commit message: Test: Disable head/tail joints to diagnose movement issue
At commit 68d721c: 8 joints controlled, robot moved
After enabling 12 joints: robot stopped moving

This commit reverts to 8-joint configuration with parameters from
working commit 68d721c to test if head/tail joints are the cause:
- Effort: 0.5 Nm for leg joints
- Damping: 0.01, Friction: 0.01
- Only 8 leg joints in controller config

Changes:
- pidog_controllers.yaml: commented out 4 head/tail joints
- pidog_gazebo_controller.py: removed head/tail from joint_names
- URDF: reverted to effort=0.5, damping=0.01, friction=0.01

If movement works with this config, we know enabling head/tail breaks it.
Next step will be to investigate WHY and fix the root cause.

File: pidog_description/urdf/pidog.urdf (robot description, URDF)
Before this commit: robot PiDog, 31 links, 30 joints
Joints:
- joint back_left_leg_b_to_a: limit lower=-1.57 upper=1.57 effort=0.15 velocity=7.0 -> lower=-1.57 upper=1.57 effort=0.5 velocity=7.0
- joint back_right_leg_b_to_a: limit lower=-1.57 upper=1.57 effort=0.15 velocity=7.0 -> lower=-1.57 upper=1.57 effort=0.5 velocity=7.0
- joint body_to_back_left_leg_b: limit lower=-1.57 upper=1.57 effort=0.15 velocity=7.0 -> lower=-1.57 upper=1.57 effort=0.5 velocity=7.0
- joint body_to_back_right_leg_b: limit lower=-1.57 upper=1.57 effort=0.15 velocity=7.0 -> lower=-1.57 upper=1.57 effort=0.5 velocity=7.0
- joint body_to_front_left_leg_b: limit lower=-1.57 upper=1.57 effort=0.15 velocity=7.0 -> lower=-1.57 upper=1.57 effort=0.5 velocity=7.0
- joint body_to_front_right_leg_b: limit lower=-1.57 upper=1.57 effort=0.15 velocity=7.0 -> lower=-1.57 upper=1.57 effort=0.5 velocity=7.0
- joint front_left_leg_b_to_a: limit lower=-1.57 upper=1.57 effort=0.15 velocity=7.0 -> lower=-1.57 upper=1.57 effort=0.5 velocity=7.0
- joint front_right_leg_b_to_a: limit lower=-1.57 upper=1.57 effort=0.15 velocity=7.0 -> lower=-1.57 upper=1.57 effort=0.5 velocity=7.0
- joint motor_8_to_tail: limit lower=-1.57 upper=1.57 effort=0.15 velocity=7.0 -> lower=-1.57 upper=1.57 effort=0.5 velocity=7.0

Commit message: Fix position_controller crash: Increase neck effort limits and reduce PID gains
Root cause: Neck joints had very low effort limits (0.14 Nm) combined with
aggressive PID gains (P=10.0). When tracking positions, the controller would
command effort far exceeding the limit:
- Position error of 0.1 rad × P gain of 10.0 = 1.0 Nm commanded
- 1.0 Nm is 7x over the 0.14 Nm limit → controller crash!

This caused the position_controller to crash immediately after activation,
leaving the robot standing but unable to move.

Fix applied:
1. Increased neck effort limits: 0.14 Nm → 0.5 Nm (match leg joints)
   - neck1_to_motor_9, neck2_to_motor_10, neck3_to_motor_11
2. Reduced neck/tail PID gains (appropriate for lighter 5g neck links):
   - P: 10.0 → 5.0 (half of leg gains)
   - D: 5.0 → 2.5
   - I: 0.3 → 0.2
   - i_clamp: 0.8 → 0.5

The neck joints are much lighter (5g links) than legs (10-13.5g) and don't
need aggressive control. The reduced gains prevent overshoot while still
providing good tracking.

Technical details:
- Neck mass: 0.005 kg per link (5g)
- Leg mass: 0.010-0.0135 kg per link (10-13.5g)
- Neck inertia: ~1-4e-6 kg·m² (very light)
- Previous effort limit (0.14 Nm) was based on light load assumption
- But with high PID gains, commanded effort exceeded limit during tracking
- New effort limit (0.5 Nm) matches legs and prevents saturation
- Reduced PID gains appropriate for actual neck dynamics

File: pidog_description/urdf/pidog.urdf (robot description, URDF)
Before this commit: robot PiDog, 31 links, 30 joints
Joints:
- joint neck1_to_motor_9: limit lower=-1.57 upper=1.57 effort=0.14 velocity=7.5 -> lower=-1.57 upper=1.57 effort=0.5 velocity=7.5
- joint neck2_to_motor_10: limit lower=-1.57 upper=1.57 effort=0.14 velocity=7.5 -> lower=-1.57 upper=1.57 effort=0.5 velocity=7.5
- joint neck3_to_motor_11: limit lower=-1.57 upper=1.57 effort=0.14 velocity=7.5 -> lower=-1.57 upper=1.57 effort=0.5 velocity=7.5

Commit message: Implement Phase 1: IMU + Contact Sensors for Fast Running
**SENSORS ADDED**:
- IMU sensor (6-DOF): 100 Hz, realistic noise (σ=0.01 rad/s, σ=0.1 m/s²)
  * Mounted on body center for balance/orientation sensing
  * Provides: roll, pitch, yaw, angular velocity, linear acceleration
- Contact sensors (4 feet): 50 Hz, binary ground contact detection
  * Back right, front right, back left, front left
  * Critical for detecting stance vs swing phase and flight phase

**URDF CHANGES** (pidog.urdf):
- Added imu_link with Gazebo IMU sensor plugin
- Added contact sensor plugins to all 4 acrylic foot pads
- Configured realistic Gaussian noise matching hardware specs

**WORLD PLUGINS** (pidog.sdf):
- Added gz-sim-imu-system plugin for IMU support
- Added gz-sim-sensors-system plugin for sensor rendering

**LAUNCH FILE** (gazebo.launch.py):
- Added ROS2 bridge for /imu topic (sensor_msgs/Imu)
- Contact sensors use native Gazebo ROS bumper plugin

**NEW RL ENVIRONMENT** (pidog_rl_env_sensors.py):
- Extended observation space: 36D → 52D
  * NEW: IMU orientation (roll, pitch, yaw) - 3D
  * NEW: IMU angular velocity - 3D
  * NEW: IMU linear acceleration - 3D
  * NEW: Foot contact sensors - 4D (binary)
  * NEW: Terrain height estimate - 1D
  * Kept: Joint states, body velocity, gait command
- Dual reward modes:
  * 'conservative': Stability-focused baseline (Phase 1)
  * 'fast_running': Speed-optimized for 2.0+ m/s (Phase 2)

**REWARD FUNCTION DESIGN** (REWARD_FUNCTION_DESIGN.md):
- Complete documentation of reward system for user review
- Speed rewards (60%): Linear + milestone bonuses at 1.2/1.8/2.2 m/s
- Stability rewards (30%): Height, orientation (roll/pitch), angular velocity
- Gait quality (10%): Flight phase detection from contact sensors
- Energy penalties (5%): Smooth motion, efficiency
- Termination: -100 penalty for falls (roll/pitch > 1.2 rad, height < 4cm)

**TUNABLE PARAMETERS** (ready for user customization):
- forward_vel_weight: 15.0 (speed priority)
- fall_penalty: -100.0 (safety)
- flight_reward: 3.0 (encourage galloping)
- pitch_tolerance: 0.6 rad (allow forward lean)
- roll_tolerance: 0.4 rad (lateral stability)

**NEXT STEPS**:
1. User reviews REWARD_FUNCTION_DESIGN.md and tunes parameters
2. Rebuild workspace and test sensors in Gazebo
3. Train Phase 1 (conservative, 50K steps) for baseline
4. Train Phase 2 (fast_running, 100K steps) for speed
5. Target: 1.5-2.0 m/s galloping with <5% fall rate

**EXPECTED PERFORMANCE**:
- Phase 1 baseline: 0.8-1.0 m/s stable trot
- Phase 2 optimized: 1.5-2.0 m/s with flight phase
- Phase 3 stretch: 2.2+ m/s maximum speed

File: pidog_description/urdf/pidog.urdf (robot description, URDF)
Before this commit: robot PiDog, 31 links, 30 joints
Links:
- added link imu_link, mass 0.001
Joints:
- added joint imu_joint: type fixed, parent body, child imu_link, origin xyz=0 0 0.02 rpy=0 0 0

Commit message: local claude

File: pidog_description/urdf/pidog.urdf (robot description, URDF)
Before this commit: robot PiDog, 32 links, 31 joints
Links:
- added link camera_link, mass 0.001; visual box size=0.005 0.01 0.005
- added link mic_center_link, mass 0.001; visual sphere radius=0.002
- added link mic_left_link, mass 0.001; visual sphere radius=0.002
- added link mic_right_link, mass 0.001; visual sphere radius=0.002
- added link rgb_led_link, mass 0.001; visual box size=0.04 0.02 0.002
- added link speaker_link, mass 0.001; visual cylinder length=0.003 radius=0.008
- added link touch_sensor_link, mass 0.001; collision box size=0.012 0.018 0.001; visual box size=0.012 0.018 0.001
- added link ultrasonic_link, mass 0.001; visual cylinder length=0.004 radius=0.008; visual cylinder length=0.004 radius=0.008
Joints:
- added joint camera_joint: type fixed, parent head, child camera_link, origin xyz=0.03 0 0.02 rpy=0 0 0
- added joint mic_center_joint: type fixed, parent head, child mic_center_link, origin xyz=0.025 0 0.025 rpy=0 0 0
- added joint mic_left_joint: type fixed, parent head, child mic_left_link, origin xyz=0.02 0.015 0.025 rpy=0 0 0
- added joint mic_right_joint: type fixed, parent head, child mic_right_link, origin xyz=0.02 -0.015 0.025 rpy=0 0 0
- added joint rgb_led_joint: type fixed, parent body, child rgb_led_link, origin xyz=0.045 0 0.01 rpy=0 0 0
- added joint speaker_joint: type fixed, parent body, child speaker_link, origin xyz=-0.03 0 -0.015 rpy=0 0 0
- added joint touch_sensor_joint: type fixed, parent head, child touch_sensor_link, origin xyz=-0.003 0 0.020 rpy=0 0 0
- added joint ultrasonic_joint: type fixed, parent head, child ultrasonic_link, origin xyz=0.0 0.0 0.036 rpy=0 0 0

Commit message: Adjust sensor positions to match hardware layout
- Move touch sensor back by 2× its length (0.024m) to sit on head piece
- Increase ultrasonic transducer spacing to 20mm (±0.010) to align with eye circles
- Keep ultrasonic sensor looking straight forward (no downward tilt)

All sensor positions now match physical PiDog layout per user feedback.

File: pidog_description/urdf/pidog.urdf (robot description, URDF)
Before this commit: robot PiDog, 40 links, 39 joints
Joints:
- joint touch_sensor_joint: origin xyz=-0.003 0 0.020 rpy=0 0 0 -> xyz=-0.027 0 0.020 rpy=0 0 0

Commit message: Adjust camera and IMU sensor positions
- Lower camera to center of nose (z=0.02 → 0.01)
- Rotate IMU 90° to lay flat on its side (rpy="0 1.5708 0")

Both sensors now match physical hardware orientation.

File: pidog_description/urdf/pidog.urdf (robot description, URDF)
Before this commit: robot PiDog, 40 links, 39 joints
Joints:
- joint camera_joint: origin xyz=0.03 0 0.02 rpy=0 0 0 -> xyz=0.03 0 0.01 rpy=0 0 0
- joint imu_joint: origin xyz=0 0 0.02 rpy=0 0 0 -> xyz=0 0 0.02 rpy=0 1.5708 0

Commit message: Move camera to front of nose laying flat
- Move forward: x=0.03 → 0.04
- Lower position: z=0.01 → 0.005
- Add pitch rotation to lay flat on nose: rpy="0 0.2 0"

Camera now sits flat at the front of the nose.

File: pidog_description/urdf/pidog.urdf (robot description, URDF)
Before this commit: robot PiDog, 40 links, 39 joints
Joints:
- joint camera_joint: origin xyz=0.03 0 0.01 rpy=0 0 0 -> xyz=0.04 0 0.005 rpy=0 0.2 0

Commit message: Lower camera and add IMU visual geometry
- Lower camera by 3× its length (z=0.005 → -0.010)
- Add MPU6050 visual representation to IMU link (21×16×3mm blue box)

Fixes "no geometry" warning for imu_link.

File: pidog_description/urdf/pidog.urdf (robot description, URDF)
Before this commit: robot PiDog, 40 links, 39 joints
Links:
- link imu_link: geometry visual box size=0.021 0.016 0.003
Joints:
- joint camera_joint: origin xyz=0.04 0 0.005 rpy=0 0.2 0 -> xyz=0.04 0 -0.010 rpy=0 0.2 0

Commit message: Remove LED strip and fix IMU position
- Remove RGB LED strip (not needed for simulation)
- Move IMU to side of body (y=0 → 0.025) instead of centered inside
- Restore IMU to original orientation (remove rotation)

IMU now matches physical PiDog placement on the side.

File: pidog_description/urdf/pidog.urdf (robot description, URDF)
Before this commit: robot PiDog, 40 links, 39 joints
Links:
- removed link rgb_led_link
Joints:
- removed joint rgb_led_joint
- joint imu_joint: origin xyz=0 0 0.02 rpy=0 1.5708 0 -> xyz=0 0.025 0.02 rpy=0 0 0

Commit message: Fix IMU position to left side surface
Changed z coordinate from 0.02 to 0 to place IMU on left side
surface (y=0.025) instead of on top of body.

File: pidog_description/urdf/pidog.urdf (robot description, URDF)
Before this commit: robot PiDog, 39 links, 38 joints
Joints:
- joint imu_joint: origin xyz=0 0.025 0.02 rpy=0 0 0 -> xyz=0 0.025 0 rpy=0 0 0

Commit message: Move IMU to left side at mid-height
Adjusted z from 0 (belly) to 0.01 to position IMU on the
left side surface at mid-height, not on the belly.

File: pidog_description/urdf/pidog.urdf (robot description, URDF)
Before this commit: robot PiDog, 39 links, 38 joints
Joints:
- joint imu_joint: origin xyz=0 0.025 0 rpy=0 0 0 -> xyz=0 0.025 0.01 rpy=0 0 0

Commit message: Move IMU to actual left side surface
Changed position from (0, 0.025, 0.01) to (0, 0.055, 0.02)
to place IMU on the actual left side surface instead of
inside the body. Body is 225mm wide, so side is at ~55mm.

File: pidog_description/urdf/pidog.urdf (robot description, URDF)
Before this commit: robot PiDog, 39 links, 38 joints
Joints:
- joint imu_joint: origin xyz=0 0.025 0.01 rpy=0 0 0 -> xyz=0 0.055 0.02 rpy=0 0 0

Commit message: Rotate IMU 90° to stand vertically on left side
Added 90° rotation around Z-axis (rpy="0 0 1.5708") so the IMU
stands vertically on the left side surface instead of laying flat.
Adjusted position to (0, 0.05, 0.01).

File: pidog_description/urdf/pidog.urdf (robot description, URDF)
Before this commit: robot PiDog, 39 links, 38 joints
Joints:
- joint imu_joint: origin xyz=0 0.055 0.02 rpy=0 0 0 -> xyz=0 0.05 0.01 rpy=0 0 1.5708

Commit message: Fix IMU rotation - rotate around Y-axis instead of Z-axis
Changed from rpy="0 0 1.5708" to rpy="0 1.5708 0" to properly
orient the IMU vertically on the left side surface.

File: pidog_description/urdf/pidog.urdf (robot description, URDF)
Before this commit: robot PiDog, 39 links, 38 joints
Joints:
- joint imu_joint: origin xyz=0 0.05 0.01 rpy=0 0 1.5708 -> xyz=0 0.05 0.01 rpy=0 1.5708 0

Commit message: Move IMU towards left legs on left face of body
Changed X position from 0 to -0.03 to position IMU near the
left legs on the left face of body, as on real hardware.

File: pidog_description/urdf/pidog.urdf (robot description, URDF)
Before this commit: robot PiDog, 39 links, 38 joints
Joints:
- joint imu_joint: origin xyz=0 0.05 0.01 rpy=0 1.5708 0 -> xyz=-0.03 0.05 0.01 rpy=0 1.5708 0

Commit message: Move IMU further back and out on left side
- Move backwards by 3× its length (x: -0.03 → -0.093)
- Move slightly more to left side to show (y: 0.05 → 0.055)

IMU now positioned near left rear legs, visible on left face.

File: pidog_description/urdf/pidog.urdf (robot description, URDF)
Before this commit: robot PiDog, 39 links, 38 joints
Joints:
- joint imu_joint: origin xyz=-0.03 0.05 0.01 rpy=0 1.5708 0 -> xyz=-0.093 0.055 0.01 rpy=0 1.5708 0

Commit message: Bring IMU out to visible left surface
Increased Y from 0.055 to 0.065 to make IMU more visible
on the left side surface.

File: pidog_description/urdf/pidog.urdf (robot description, URDF)
Before this commit: robot PiDog, 39 links, 38 joints
Joints:
- joint imu_joint: origin xyz=-0.093 0.055 0.01 rpy=0 1.5708 0 -> xyz=-0.093 0.065 0.01 rpy=0 1.5708 0

Commit message: Fix IMU axes - place on left side near back legs
Corrected coordinate system understanding:
- X = 0.065 (left side, was negative)
- Y = -0.03 (towards back, was positive)
- Z = 0.01 (mid-height)

IMU now correctly positioned on left face near back legs.

File: pidog_description/urdf/pidog.urdf (robot description, URDF)
Before this commit: robot PiDog, 39 links, 38 joints
Joints:
- joint imu_joint: origin xyz=-0.093 0.065 0.01 rpy=0 1.5708 0 -> xyz=0.065 -0.03 0.01 rpy=0 1.5708 0

Commit message: fix x

File: pidog_description/urdf/pidog.urdf (robot description, URDF)
Before this commit: robot PiDog, 39 links, 38 joints
Joints:
- joint imu_joint: origin xyz=0.065 -0.03 0.01 rpy=0 1.5708 0 -> xyz=0.032 -0.03 0.01 rpy=0 1.5708 0
